File: Keyboard/hardware/sonic-rec9388-keyboard.kicad_pcb (KiCad board)
At the start: 2 copper layers, 367 x 134.6 mm, 114 parts, among them J1 To main board, Q1 NPN, SW1 RESET, U1 74LS145, U2 74LS161, U3 4021

Commit message: Fix reset capacitor polarity
Parts:
- moved C1 2.48 mm to (-7.24, -122.2), turned to -90 degrees
Connections:
- C1 pad 1: GND -> RESET
- C1 pad 2: RESET -> GND
