File: Keyboard/hardware/sonic-rec9388-keyboard.kicad_sch (KiCad schematic)
At the start: 114 parts, among them J1 To main board, Q1 NPN, SW1 RESET, U1 74LS145, U2 74LS161, U3 4021

Commit message: Fix reset capacitor polarity
Connections:
- net GND: now also C1.2; no longer C1.1
- net RESET: now also C1.1; no longer C1.2
Other:
- moved on the sheet: C1
Changed lines of the file:
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@@
 	)
 	(junction
-		(at 200.66 135.89)
-		(diameter 0)
-		(color 0 0 0 0)
-	)
-	(junction
 		(at 63.5 147.32)
 		(diameter 0)
@@
 	)
 	(junction
+		(at 200.66 135.89)
+		(diameter 0)
+		(color 0 0 0 0)
+	)
+	(junction
 		(at 62.865 29.845)
 		(diameter 0)
@@
 	(wire
 		(pts
-			(xy 200.66 135.89) (xy 201.93 135.89)
-		)
-		(stroke
-			(width 0)
-			(type default)
-		)
-	)
-	(wire
-		(pts
 			(xy 97.79 76.835) (xy 97.79 87.63)
 		)
@@
 	(wire
 		(pts
+			(xy 200.66 135.89) (xy 201.93 135.89)
+		)
+		(stroke
+			(width 0)
+			(type default)
+		)
+	)
+	(wire
+		(pts
 			(xy 46.99 140.97) (xy 50.8 140.97)
 		)
@@
 	(symbol
 		(lib_id "Device:C_Polarized")
-		(at 200.66 139.7 180)
+		(at 200.66 139.7 0)
 		(unit 1)
 		(exclude_from_sim no)
@@
 		(dnp no)
 		(property "Reference" "C1"
-			(at 204.47 139.3189 0)
+			(at 196.85 140.0811 0)
 			(effects
 				(font
@@
 		)
 		(property "Value" "C_Polarized"
-			(at 204.47 141.8589 0)
+			(at 196.85 137.5411 0)
 			(effects
 				(font
@@
 		)
 		(property "Footprint" "Capacitor_THT:CP_Radial_D5.0mm_P2.50mm"
-			(at 199.6948 135.89 0)
+			(at 201.6252 143.51 0)
 			(effects
 				(font
